File: UnderwaterGlider/MainControl.kicad_sch (KiCad schematic)
At the start: 110 parts, among them J1 Micro_SD_Card_Det1, J2 Conn_01x02, J22 SBus, J3 Conn_01x04_MountingPin, J4 Conn_01x04_MountingPin, J5 Conn_01x02, J6 Conn_01x03, J7 Conn_01x03, J8 Conn_01x03, J9 Conn_01x03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

Commit message: update layout
Parts:
- J1: footprint (none) -> UnderwaterGlider:TF-SMD_TF-PUSH
- U2: footprint RM24:PQFN50P300X250X97-14N -> 0_RM2024:PQFN50P300X250X97-14N
Changed lines of the file:
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@@
 			)
 		)
-		(property "Footprint" "RM24:PQFN50P300X250X97-14N"
+		(property "Footprint" "0_RM2024:PQFN50P300X250X97-14N"
 			(at 322.58 138.43 0)
 			(effects
@@
 			)
 		)
-		(property "Footprint" ""
+		(property "Footprint" "UnderwaterGlider:TF-SMD_TF-PUSH"
 			(at 391.16 21.59 0)
 			(effects
