File: UnderwaterGlider/MainControl.kicad_sch (KiCad schematic)
At the start: 137 parts, among them J1 Micro_SD_Card_Det1, J11 Conn_01x02_MountingPin, J12 Conn_01x02_MountingPin, J13 Conn_01x02_MountingPin, J14 Conn_01x02_MountingPin, J15 Conn_01x02_MountingPin, J16 Conn_01x02_MountingPin, J17 Conn_01x02_MountingPin, J18 Conn_01x02_MountingPin, J19 Conn_01x04_MountingPin, J2 Conn_01x02, J20 Conn_01x04, J22 SBus, J28 SWD, J3 Conn_01x04_MountingPin, J4 Conn_01x04_MountingPin, J5 Conn_01x02, J6 Conn_01x03, J7 Conn_01x03, J8 Conn_01x03, J9 Conn_01x03, SW1 NRST, SW2 BOOT0, U1 STM32H743VITx, U13 SN75176AD, U14 SN75176AD, U15 SN75176AD, U16 CH343P, U2 ICM-42688-P, U4 TJA1042T-3, U5 SN75179B, U6 TPD4E1U06DCKR, Y1 25MHz

Commit message: update layout
Parts:
- removed RN19: 82R, Resistor_SMD:R_Array_Concave_4x0603, symbol Device:R_Pack04
Connections:
- net CAN1_H: now also J11.2 (Pin_2), J12.2 (Pin_2); no longer J11.1 (Pin_1), J12.1 (Pin_1)
- net CAN1_L: now also J11.1 (Pin_1), J12.1 (Pin_1); no longer J11.2 (Pin_2), J12.2 (Pin_2)
- net CAN1_RX: now also RN6.7 (R2.2); no longer RN6.6 (R3.2)
- net CAN1_TX: now also RN6.8 (R1.2); no longer RN6.7 (R2.2)
- net Dir+: now also J3.2 (Pin_2); no longer J3.3 (Pin_3)
- net Dir-: now also J3.1 (Pin_1); no longer J3.4 (Pin_4)
- net GND: now also RN12.1 (R1.1), RN12.2 (R2.1), RN12.7 (R2.2), RN12.8 (R1.2); no longer RN12.3 (R3.1), RN12.4 (R4.1), RN12.5 (R4.2), RN12.6 (R3.2), RN6.1 (R1.1), RN6.4 (R4.1), RN6.5 (R4.2), RN6.8 (R1.2)
- net PA13: now also RN6.4 (R4.1)
- net PA14: now also RN6.3 (R3.1)
- net PD0: now also RN6.2 (R2.1); no longer RN6.3 (R3.1)
- net PD1: now also RN6.1 (R1.1); no longer RN6.2 (R2.1)
- net PE0: now also RN14.2 (R2.1); no longer RN14.1 (R1.1)
- net PE1: now also RN14.1 (R1.1); no longer RN14.2 (R2.1)
- net PE7: now also RN12.4 (R4.1); no longer RN12.2 (R2.1)
- net PE8: now also RN12.3 (R3.1); no longer RN12.1 (R1.1)
- net Pul+: now also J3.4 (Pin_4); no longer J3.1 (Pin_1)
- net Pul-: now also J3.3 (Pin_3); no longer J3.2 (Pin_2)
- net SWD_CLK: now also RN6.6 (R3.2)
- net SWD_DIO: now also RN6.5 (R4.2)
- net TIM2_CH3: no longer RN18.6 (R3.2)
- net TIM2_CH4: no longer RN18.8 (R1.2)
- net TIM4_CH3: now also RN18.6 (R3.2)
- net TIM4_CH4: now also RN18.8 (R1.2)
- net UART7_RX: now also RN12.5 (R4.2); no longer RN12.7 (R2.2)
- net UART7_TX: now also RN12.6 (R3.2); no longer RN12.8 (R1.2)
- net UART8_RX: now also RN14.8 (R1.2); no longer RN14.7 (R2.2)
- net UART8_TX: now also RN14.7 (R2.2); no longer RN14.8 (R1.2)
