File: UnderwaterGlider/Power.kicad_sch (KiCad schematic)
At the start: 187 parts, among them J10 Conn_01x02, Q1 BSC070N10, Q2 BSC070N10, U10 RS3236, U11 RS3236, U12 LMR51610, U17 RY3430, U18 LM5145, U19 TPS54560BDDA, U3 LT3042EMSE(TOKMAS)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

Commit message: update layout
Parts:
- removed C120, C121, C122, C86: 47u, symbol Device:C_Polarized
- C21, C22, C23, C47, C48, C49, C84, C85: footprint (none) -> Capacitor_THT:CP_Radial_D6.3mm_P2.50mm
- F1: footprint (none) -> Fuse:Fuseholder_Littelfuse_Nano2_157x
Connections:
- net VIN is gone; now on net +48V: U12.4 (EN), U12.5 (IN)
- net +12V_Motor: now also C84.1, C85.1
- net +5V: no longer C23.1
- net +5V_SatellieCom: now also C23.1; no longer C47.1, C49.1
- net 7.4v_Servo: now also C47.1, C49.1; no longer C84.1, C85.1
- net GND: now also J10.1 (Pin_1); no longer J10.2 (Pin_2)
- net at F1.1: now also J10.2 (Pin_2); no longer J10.1 (Pin_1)
Other:
- moved on the sheet: J10

Commit message: update placement
Parts:
- added J21: Conn_01x02, Connector_AMASS:AMASS_XT30PW-F_1x02_P2.50mm_Horizontal, symbol Connector_Generic:Conn_01x02
- L1, L4, L5, L8: footprint Inductor_SMD:L_Changjiang_FXL1770 -> Inductor_SMD:L_Sunlord_MWSA0603S
Connections:
- net VOUT is gone; now on net +24V: R46.1, R47.1
- net +24V: now also J21.2 (Pin_2)
- net GND: now also J21.1 (Pin_1)
- net 7.4v_Servo renamed +7.4v_Servo
