File: UnderwaterGlider/UnderwaterGlider.kicad_pcb (KiCad board)
At the start: 2 copper layers, 118 parts, among them J10 Conn_01x02, J2 Conn_01x02, J22 SBus, J3 Conn_01x04_MountingPin, J4 Conn_01x04_MountingPin, J5 Conn_01x02, J6 Conn_01x03, J7 Conn_01x03, J8 Conn_01x03, J9 Conn_01x03, SW1 NRST, SW2 BOOT0, U1 STM32H743VITx, U13 SN75176AD, U14 SN75176AD, U15 SN75176AD, U16 CH343P, U3 LT3042xMSE, U4 TJA1042T-3, U5 SN75179B, U6 TPD4E1U06DCKR, U7 TPS54560BDDA, Y1 25MHz

Commit message: update layout
Parts:
- added C100: C, Capacitor_SMD:C_1206_3216Metric, F.Cu at (190.0, -13.3)
- added C101: C, Capacitor_SMD:C_1210_3225Metric, B.Cu at (63.9, 3.93)
- added C102: C, Capacitor_SMD:C_1206_3216Metric, F.Cu at (190.0, -9.96)
- added C103: C, Capacitor_SMD:C_1210_3225Metric, B.Cu at (67.1, 3.96)
- added C104: C, Capacitor_SMD:C_1206_3216Metric, F.Cu at (190.0, -6.61)
- added C105: C, Capacitor_SMD:C_1210_3225Metric, B.Cu at (70.3, 3.96)
- added C106: C, Capacitor_SMD:C_1206_3216Metric, F.Cu at (190.0, -3.26)
- added C107: C, Capacitor_SMD:C_1206_3216Metric, F.Cu at (190.0, 0.09)
- added C108: 100uF 63V, Capacitor_THT:CP_Radial_D8.0mm_P3.50mm, B.Cu at (54.8, 2.15)
- added C109: 220uF 35V, Capacitor_THT:CP_Radial_D8.0mm_P3.50mm, F.Cu at (160.9, -54.9)
- added C110: 100uF 63V, Capacitor_THT:CP_Radial_D8.0mm_P3.50mm, B.Cu at (46.2, 2.15)
- added C111: 220uF 35V, Capacitor_THT:CP_Radial_D8.0mm_P3.50mm, F.Cu at (160.9, -35.8)
- added C112: 10u, Capacitor_SMD:C_1206_3216Metric, F.Cu at (186.5, 93.6)
- added C113: 10u, Capacitor_SMD:C_1206_3216Metric, F.Cu at (192.1, 73.5)
- added C114: 10u, Capacitor_SMD:C_1206_3216Metric, F.Cu at (192.1, 76.8)
- added C115: 4.7n, Capacitor_SMD:C_0603_1608Metric, F.Cu at (173.9, 52.4)
- added C116: 47p, Capacitor_SMD:C_0603_1608Metric, F.Cu at (173.9, 54.9)
- added C117: 100n, Capacitor_SMD:C_0603_1608Metric, F.Cu at (178.0, 22.2)
- added C118: 10u, Capacitor_SMD:C_1206_3216Metric, F.Cu at (192.1, 80.2)
- added C119: 10u, Capacitor_SMD:C_1206_3216Metric, F.Cu at (192.1, 83.5)
- added C14: 10u, Capacitor_SMD:C_1206_3216Metric, F.Cu at (175.2, 73.5)
- added C15: 10u, Capacitor_SMD:C_1206_3216Metric, F.Cu at (175.2, 76.8)
- added C19: 47u, Capacitor_Tantalum_SMD:CP_EIA-3216-18_Kemet-A_Pad1.58x1.35mm_HandSolder, F.Cu at (202.3, 52.9)
- added C2: 47p, Capacitor_SMD:C_0603_1608Metric, F.Cu at (165.9, 24.7)
- added C21: 47u, Capacitor_THT:CP_Radial_D6.3mm_P2.50mm, F.Cu at (166.7, 60.0)
- added C22: 47u, Capacitor_THT:CP_Radial_D6.3mm_P2.50mm, F.Cu at (166.7, 67.9)
- added C23: 47u, Capacitor_THT:CP_Radial_D6.3mm_P2.50mm, F.Cu at (174.7, 60.0)
- added C24: 4.7n, Capacitor_SMD:C_0603_1608Metric, F.Cu at (165.9, 29.8)
- added C25: 47p, Capacitor_SMD:C_0603_1608Metric, F.Cu at (165.9, 32.3)
- added C26: 100n, Capacitor_SMD:C_0603_1608Metric, F.Cu at (165.9, 34.8)
- added C28: 10u, Capacitor_SMD:C_1206_3216Metric, F.Cu at (175.2, 80.2)
- added C3: 4.7n, Capacitor_SMD:C_0603_1608Metric, F.Cu at (165.9, 27.2)
- added C32: 10u, Capacitor_SMD:C_1206_3216Metric, F.Cu at (175.2, 93.6)
- added C33: 10u, Capacitor_SMD:C_1206_3216Metric, F.Cu at (180.8, 73.5)
- added C34: 10u, Capacitor_SMD:C_1206_3216Metric, F.Cu at (180.8, 76.8)
- added C35: 10u, Capacitor_SMD:C_1206_3216Metric, F.Cu at (180.8, 80.2)
- added C36: 10u, Capacitor_SMD:C_0603_1608Metric, F.Cu at (165.9, 37.3)
- added C37: 100n, Capacitor_SMD:C_0603_1608Metric, F.Cu at (165.9, 39.8)
- added C38: 10n, Capacitor_SMD:C_0603_1608Metric, F.Cu at (165.9, 42.3)
- added C39: 10u, Capacitor_SMD:C_0603_1608Metric, F.Cu at (165.9, 44.8)
- added C40: 100n, Capacitor_SMD:C_0603_1608Metric, F.Cu at (165.9, 47.3)
- added C41: 10u, Capacitor_SMD:C_0603_1608Metric, F.Cu at (165.9, 49.8)
- added C42: 100n, Capacitor_SMD:C_0603_1608Metric, F.Cu at (165.9, 52.4)
- added C43: 10n, Capacitor_SMD:C_0603_1608Metric, F.Cu at (165.9, 54.9)
- added C44: 10u, Capacitor_SMD:C_0603_1608Metric, F.Cu at (169.9, 22.2)
- added C45: 100n, Capacitor_SMD:C_0603_1608Metric, F.Cu at (169.9, 24.7)
- added C47: 47u, Capacitor_THT:CP_Radial_D6.3mm_P2.50mm, F.Cu at (174.7, 67.9)
- added C48: 47u, Capacitor_THT:CP_Radial_D6.3mm_P2.50mm, F.Cu at (182.7, 60.0)
- added C49: 47u, Capacitor_THT:CP_Radial_D6.3mm_P2.50mm, F.Cu at (182.7, 67.9)
- added C50: 20p, Capacitor_SMD:C_0603_1608Metric, F.Cu at (169.9, 27.2)
- added C51: 10u, Capacitor_SMD:C_0603_1608Metric, F.Cu at (169.9, 29.8)
- added C53: 10u, Capacitor_SMD:C_0603_1608Metric, F.Cu at (169.9, 32.3)
- added C63: 10u, Capacitor_SMD:C_0603_1608Metric, F.Cu at (169.9, 34.8)
- added C64: 10u, Capacitor_SMD:C_0603_1608Metric, F.Cu at (169.9, 37.3)
- added C65: 10u, Capacitor_SMD:C_0603_1608Metric, F.Cu at (169.9, 39.8)
- added C66: 10u, Capacitor_SMD:C_0603_1608Metric, F.Cu at (169.9, 42.3)
- added C67: 100n, Capacitor_SMD:C_0603_1608Metric, F.Cu at (169.9, 44.8)
- added C68: 10u, Capacitor_SMD:C_0603_1608Metric, F.Cu at (169.9, 47.3)
- added C69: 100n, Capacitor_SMD:C_0603_1608Metric, F.Cu at (169.9, 49.8)
- added C74: 4.7u, Capacitor_SMD:C_0603_1608Metric, F.Cu at (169.9, 52.4)
- added C75: 10u, Capacitor_SMD:C_1206_3216Metric, F.Cu at (180.8, 83.5)
- added C77: 10u, Capacitor_SMD:C_1206_3216Metric, F.Cu at (180.8, 86.9)
- added C78: 10u, Capacitor_SMD:C_1206_3216Metric, F.Cu at (180.8, 90.2)
- added C79: 4.7n, Capacitor_SMD:C_0603_1608Metric, F.Cu at (169.9, 54.9)
- added C80: 47p, Capacitor_SMD:C_0603_1608Metric, F.Cu at (173.9, 22.2)
- added C81: 100n, Capacitor_SMD:C_0603_1608Metric, F.Cu at (173.9, 24.7)
- added C82: 10u, Capacitor_SMD:C_1206_3216Metric, F.Cu at (180.8, 93.6)
- added C83: 10u, Capacitor_SMD:C_1206_3216Metric, F.Cu at (186.5, 73.5)
- added C84: 47u, Capacitor_THT:CP_Radial_D6.3mm_P2.50mm, F.Cu at (190.7, 60.0)
- added C85: 47u, Capacitor_THT:CP_Radial_D6.3mm_P2.50mm, F.Cu at (190.7, 67.9)
- added C87: 270p, Capacitor_SMD:C_0603_1608Metric, F.Cu at (177.5, -62.9)
- added C88: 5.6p, Capacitor_SMD:C_0603_1608Metric, F.Cu at (177.5, -60.4)
- added C89: 330p, Capacitor_SMD:C_0603_1608Metric, F.Cu at (177.5, -57.9)
- added C90: 100n, Capacitor_SMD:C_0603_1608Metric, F.Cu at (45.6, -8.95)
- added C91: 470n, Capacitor_SMD:C_0603_1608Metric, F.Cu at (177.5, -52.9)
- added C92: 100n, Capacitor_SMD:C_0603_1608Metric, F.Cu at (177.5, -50.4)
- added C93: 22u, Capacitor_SMD:C_0805_2012Metric, F.Cu at (54.2, -5.14)
- added C94: 22u, Capacitor_SMD:C_0805_2012Metric, F.Cu at (52.2, -5.14)
- added C95: 8.2p, Capacitor_SMD:C_0603_1608Metric, F.Cu at (177.5, -47.8)
- added C96: 100nF, Capacitor_SMD:C_0603_1608Metric, F.Cu at (177.5, -45.3)
- added C97: 2.2u, Capacitor_SMD:C_0603_1608Metric, F.Cu at (63.0, -9.50)
- added C98: 100n, Capacitor_SMD:C_0603_1608Metric, F.Cu at (81.1, -64.1)
- added C99: C, Capacitor_SMD:C_1210_3225Metric, B.Cu at (60.7, 3.96)
- added D12: LED, LED_SMD:LED_0603_1608Metric, F.Cu at (37.0, -11.7)
- added D13: SMCJ28A, Diode_SMD:D_SMC, F.Cu at (201.3, 67.7)
- added D14: ST20100L, RM25:D_PowerDI-5, F.Cu at (199.3, 91.5)
- added D15: SMAJ5.0A, Diode_SMD:D_SMA, F.Cu at (158.3, 61.5)
- added D16: SMF3.3v, Diode_SMD:D_SMF, F.Cu at (212.5, 46.0)
- added D17: SMF3.3v, Diode_SMD:D_SMF, F.Cu at (212.5, 49.4)
- added D18: SMF3.3v, Diode_SMD:D_SMF, F.Cu at (212.5, 52.8)
- added D19: SMAJ5.0A, Diode_SMD:D_SMA, F.Cu at (158.3, 66.0)
- added D20: SMAJ7.5A, Diode_SMD:D_SMA, F.Cu at (158.3, 70.5)
- added D21: SMAJ12A, Diode_SMD:D_SMA, F.Cu at (158.3, 75.1)
- added D22: LED, LED_SMD:LED_0603_1608Metric, F.Cu at (205.7, 96.8)
- added D23: LED, LED_SMD:LED_0603_1608Metric, F.Cu at (205.7, 99.4)
- added D24: LED, LED_SMD:LED_0603_1608Metric, F.Cu at (209.8, 91.6)
- added D25: LED, LED_SMD:LED_0603_1608Metric, F.Cu at (209.8, 94.2)
- added D26: LED, LED_SMD:LED_0603_1608Metric, F.Cu at (209.8, 96.8)
- added D27: LED, LED_SMD:LED_0603_1608Metric, F.Cu at (209.8, 99.4)
- added D28: LED, LED_SMD:LED_0603_1608Metric, F.Cu at (213.8, 91.6)
- added D29: LED, LED_SMD:LED_0603_1608Metric, F.Cu at (213.8, 94.2)
- added D30: LED, LED_SMD:LED_0603_1608Metric, F.Cu at (213.8, 96.8)
- added D31: LED, LED_SMD:LED_0603_1608Metric, F.Cu at (213.8, 99.4)
- added D4: ST20100L, RM25:D_PowerDI-5, F.Cu at (199.3, 80.2)
- added D5: ST20100L, RM25:D_PowerDI-5, F.Cu at (199.3, 85.8)
- added D6: LED, LED_SMD:LED_0603_1608Metric, F.Cu at (209.3, 1.46)
- added D7: K34, Diode_SMD:D_SMF, F.Cu at (53.6, -8.04)
- added F1: Fuse, Fuse:Fuseholder_Littelfuse_Nano2_157x, F.Cu at (20.1, 49.9)
- added F2: Fuse, Fuse:Fuse_Littelfuse-NANO2-451_453, B.Cu at (40.1, 0.20)
- added J1: Micro_SD_Card_Det1, UnderwaterGlider:TF-SMD_TF-PUSH, F.Cu at (240.6, 51.4)
- added L1: 7.2u, Inductor_SMD:L_Changjiang_FXL1770, F.Cu at (144.3, 30.4)
- added L3: 4u7, Inductor_SMD:L_Sunlord_MWSA0402S, F.Cu at (212.2, 74.7)
- added L4: 7.2u, Inductor_SMD:L_Changjiang_FXL1770, F.Cu at (144.3, 49.2)
- added L5: 7.2u, Inductor_SMD:L_Changjiang_FXL1770, F.Cu at (144.3, 68.0)
- added L6: 10u, Inductor_SMD:L_Sunlord_MWSA0402S, F.Cu at (48.3, -5.84)
- added L7: 10u, RM25:PQ2014_10uH, F.Cu at (77.8, -13.2)
- added L8: 7.2u, Inductor_SMD:L_Changjiang_FXL1770, F.Cu at (35.3, 73.4)
- added Q1: BSC070N10, Package_TO_SOT_SMD:TDSON-8-1, B.Cu at (74.8, 1.35)
- added Q2: BSC070N10, Package_TO_SOT_SMD:TDSON-8-1, B.Cu at (68.4, -1.29)
- added R34: 16.9k, Resistor_SMD:R_0603_1608Metric, F.Cu at (178.0, 27.2)
- added R35: 47k, Resistor_SMD:R_0603_1608Metric, F.Cu at (178.0, 29.8)
- added R36: 10k, Resistor_SMD:R_0603_1608Metric, F.Cu at (178.0, 32.3)
- added R37: 16.9k, Resistor_SMD:R_0603_1608Metric, F.Cu at (178.0, 34.8)
- added R38: 243k, Resistor_SMD:R_0603_1608Metric, F.Cu at (178.0, 37.3)
- added R39: 53.6k, Resistor_SMD:R_0603_1608Metric, F.Cu at (178.0, 39.8)
- added R40: 10k, Resistor_SMD:R_0603_1608Metric, F.Cu at (178.0, 42.3)
- added R41: 47k, Resistor_SMD:R_0603_1608Metric, F.Cu at (178.0, 44.8)
- added R42: 10k, Resistor_SMD:R_0603_1608Metric, F.Cu at (178.0, 47.3)
- added R43: 33k, Resistor_SMD:R_0603_1608Metric, F.Cu at (178.0, 49.8)
- added R44: 16.9k, Resistor_SMD:R_0603_1608Metric, F.Cu at (178.0, 52.4)
- added R45: 243k, Resistor_SMD:R_0603_1608Metric, F.Cu at (178.0, 54.9)
- added R46: 3830R, Resistor_SMD:R_0603_1608Metric, F.Cu at (185.5, -67.9)
- added R47: 300k, Resistor_SMD:R_0603_1608Metric, F.Cu at (185.5, -65.4)
- added R48: 10k, Resistor_SMD:R_0603_1608Metric, F.Cu at (185.5, -62.9)
- added R49: 309k, Resistor_SMD:R_0603_1608Metric, F.Cu at (185.5, -60.4)
- added R50: 10k, Resistor_SMD:R_0603_1608Metric, F.Cu at (185.5, -57.9)
- added R51: 51k, Resistor_SMD:R_0603_1608Metric, F.Cu at (185.5, -55.4)
- added R52: 4k7, Resistor_SMD:R_0603_1608Metric, F.Cu at (185.5, -52.9)
- added R53: 4k7, Resistor_SMD:R_0603_1608Metric, F.Cu at (185.5, -50.4)
- added R54: 118k, Resistor_SMD:R_0603_1608Metric, F.Cu at (42.8, -9.67)
- added R55: 10K, Resistor_SMD:R_0603_1608Metric, F.Cu at (41.3, -8.14)
- added R56: 10k, Resistor_SMD:R_0603_1608Metric, F.Cu at (185.5, -42.8)
- added R57: NC, Resistor_SMD:R_0603_1608Metric, F.Cu at (185.5, -40.3)
- added R62: 10k, Resistor_SMD:R_0603_1608Metric, F.Cu at (185.5, -37.8)
- added R63: 560R, Resistor_SMD:R_0603_1608Metric, F.Cu at (176.9, -37.5)
- added R64: 10k, Resistor_SMD:R_0603_1608Metric, F.Cu at (40.0, -11.7)
- added R65: 0R, Resistor_SMD:R_0603_1608Metric, F.Cu at (189.5, -65.4)
- added R66: 0R, Resistor_SMD:R_0603_1608Metric, F.Cu at (189.5, -62.9)
- added R67: 16.9k, Resistor_SMD:R_0603_1608Metric, F.Cu at (186.0, 29.8)
- added R68: 243k, Resistor_SMD:R_0603_1608Metric, F.Cu at (186.0, 32.3)
- added R69: 53.6k, Resistor_SMD:R_0603_1608Metric, F.Cu at (186.0, 34.8)
- added R70: 10k, Resistor_SMD:R_0603_1608Metric, F.Cu at (186.0, 37.3)
- added R71: 82.5k, Resistor_SMD:R_0603_1608Metric, F.Cu at (186.0, 39.8)
- added R72: 10k, Resistor_SMD:R_0603_1608Metric, F.Cu at (186.0, 42.3)
- added R73: 140k, Resistor_SMD:R_0603_1608Metric, F.Cu at (186.0, 44.8)
- added R74: 10k, Resistor_SMD:R_0603_1608Metric, F.Cu at (186.0, 47.3)
- added R75: 100k, Resistor_SMD:R_0603_1608Metric, F.Cu at (186.0, 49.8)
- added R76: 51k, Resistor_SMD:R_0603_1608Metric, F.Cu at (186.0, 52.4)
- added R77: 10k, Resistor_SMD:R_0603_1608Metric, F.Cu at (186.0, 54.9)
- added R78: 10k, Resistor_SMD:R_0603_1608Metric, F.Cu at (190.0, 22.2)
- added R79: 1k, Resistor_SMD:R_0603_1608Metric, F.Cu at (190.0, 24.7)
- added R80: 1k, Resistor_SMD:R_0603_1608Metric, F.Cu at (190.0, 27.2)
- added R81: 1k, Resistor_SMD:R_0603_1608Metric, F.Cu at (190.0, 29.8)
- added R82: 1k, Resistor_SMD:R_0603_1608Metric, F.Cu at (190.0, 32.3)
- added R83: 10k, Resistor_SMD:R_0603_1608Metric, F.Cu at (190.0, 34.8)
- added R84: 10k, Resistor_SMD:R_0603_1608Metric, F.Cu at (190.0, 37.3)
- added U10: RS3236, Package_TO_SOT_SMD:SOT-23-5, F.Cu at (206.2, 74.2)
- added U11: RS3236, Package_TO_SOT_SMD:SOT-23-5, F.Cu at (206.2, 78.8)
- added U12: LMR51610, Package_TO_SOT_SMD:SOT-23-6, F.Cu at (43.7, -6.08)
- added U17: RY3430, Package_TO_SOT_SMD:SOT-23-5, F.Cu at (206.2, 88.1)
- added U18: LM5145, Package_DFN_QFN:Texas_RGY_R-PVQFN-N20_EP2.05x3.05mm, B.Cu at (60.0, -7.85)
- added U19: TPS54560BDDA, Package_SO:Texas_R-PDSO-G8_EP2.95x4.9mm_Mask2.4x3.1mm_ThermalVias, F.Cu at (168.1, 94.9)
- added U2: ICM-42688-P, 0_RM2024:PQFN50P300X250X97-14N, F.Cu at (52.2, 97.3)
- added U8: TPS54560BDDA, Package_SO:Texas_R-PDSO-G8_EP2.95x4.9mm_Mask2.4x3.1mm_ThermalVias, F.Cu at (168.1, 81.8)
- added U9: TPS54560BDDA, Package_SO:Texas_R-PDSO-G8_EP2.95x4.9mm_Mask2.4x3.1mm_ThermalVias, F.Cu at (168.1, 88.3)
- U3: value LT3042xMSE -> LT3042EMSE(TOKMAS)
- moved U16 166.7 mm to (188.0, 151.3)
- moved D11 142.2 mm to (178.1, 150.0)
- moved J10 141.1 mm to (17.8, 64.0), turned to 90 degrees
- moved U13 138.6 mm to (162.7, 119.2)
- moved U14 138.6 mm to (162.7, 125.8)
- moved U15 138.6 mm to (162.7, 132.3)
- moved U4 138.6 mm to (162.7, 106.0)
- moved D1 136.9 mm to (169.4, 138.0)
- moved D10 136.9 mm to (169.4, 151.8)
- moved D8 136.9 mm to (169.4, 142.6)
- moved D9 136.9 mm to (169.4, 147.2)
- moved Y1 129.2 mm to (188.0, 156.2)
- moved RN8 118.2 mm to (185.6, 105.1)
- moved RN9 118.2 mm to (189.8, 105.1)
- moved U5 118.0 mm to (162.7, 112.6)
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Connections:
- C27 pad 1: 3V3_IO -> +3.3V_IO
- C4 pad 1: 3V3_IMU -> +3.3V_IMU
- C46 pad 1: 3V3_IO -> +3.3V_IO
- J10 pad 1: Net-(J10-Pin_1) -> GND
- J10 pad 2: GND -> Net-(J10-Pin_2)
- R22 pad 1: 3V3_IO -> +3.3V_IO
- U16 pad 1: 3V3_IO -> +3.3V_IO
- U16 pad 3: 3V3_IO -> +3.3V_IO
- U16 pad 6: 3V3_IO -> +3.3V_IO
- U3 pad 1: Net-(U3-IN-Pad1) -> +5V
- U3 pad 10: unconnected-(U3-OUT-Pad10) -> +3.3V_SatellieCom
- U3 pad 11: Net-(U3-GND-Pad11) -> GND
- U3 pad 2: Net-(U3-IN-Pad1) -> +5V
- U3 pad 3: unconnected-(U3-EN/UV-Pad3) -> +5V
- U3 pad 4: unconnected-(U3-PG-Pad4) -> /Power/PG_SATCom_3.3v
- U3 pad 5: unconnected-(U3-ILIM-Pad5) -> GND
- U3 pad 6: unconnected-(U3-PGFB-Pad6) -> Net-(U3-PGFB)
- U3 pad 7: unconnected-(U3-SET-Pad7) -> Net-(U3-SET)
- U3 pad 8: Net-(U3-GND-Pad11) -> GND
- U3 pad 9: unconnected-(U3-OUTS-Pad9) -> +3.3V_SatellieCom
- U7 pad 6: unconnected-(U7-COMP-Pad6) -> Net-(U7-COMP)
Other:
- board outline added: 100 x 100 mm

Commit message: update placement
Parts:
- added C120: 10u, Capacitor_SMD:C_0603_1608Metric, F.Cu at (20.5, 38.5)
- added C121: 10u, Capacitor_SMD:C_0603_1608Metric, F.Cu at (87.3, 96.8)
- added C86: 10u, Capacitor_SMD:C_0603_1608Metric, F.Cu at (19.9, 27.7)
- added D32: LED, LED_SMD:LED_0603_1608Metric, F.Cu at (103.5, 91.3)
- added D33: LED, LED_SMD:LED_0603_1608Metric, F.Cu at (103.5, 100.7)
- added D34: 3V3 TVS, Diode_SMD:D_SMF, F.Cu at (93.3, 95.8)
- added D35: K34, Diode_SMD:D_SMF, F.Cu at (90.0, 95.8)
- added F3: 1.2A, Fuse:Fuse_1210_3225Metric, F.Cu at (15.8, 66.0)
- added H1: MountingHole_Pad_MP, MountingHole:MountingHole_3.2mm_M3_Pad_Via, F.Cu at (14.0, 14.0)
- added H2: MountingHole_Pad_MP, MountingHole:MountingHole_3.2mm_M3_Pad_Via, F.Cu at (14.0, 106.0)
- added H3: MountingHole_Pad_MP, MountingHole:MountingHole_3.2mm_M3_Pad_Via, F.Cu at (106.0, 106.0)
- added H4: MountingHole_Pad_MP, MountingHole:MountingHole_3.2mm_M3_Pad_Via, F.Cu at (106.0, 14.0)
- added J11: Conn_01x02_MountingPin, Connector_JST:JST_GH_SM02B-GHS-TB_1x02-1MP_P1.25mm_Horizontal, F.Cu at (73.6, 106.2)
- added J12: Conn_01x02_MountingPin, Connector_JST:JST_GH_SM02B-GHS-TB_1x02-1MP_P1.25mm_Horizontal, F.Cu at (80.6, 106.2)
- added J13: Conn_01x02_MountingPin, Connector_JST:JST_GH_SM02B-GHS-TB_1x02-1MP_P1.25mm_Horizontal, F.Cu at (58.1, 106.4)
- added J14: Conn_01x02_MountingPin, Connector_JST:JST_GH_SM02B-GHS-TB_1x02-1MP_P1.25mm_Horizontal, F.Cu at (51.1, 106.4)
- added J15: Conn_01x02_MountingPin, Connector_JST:JST_GH_SM02B-GHS-TB_1x02-1MP_P1.25mm_Horizontal, F.Cu at (42.6, 15.4)
- added J16: Conn_01x02_MountingPin, Connector_JST:JST_GH_SM02B-GHS-TB_1x02-1MP_P1.25mm_Horizontal, F.Cu at (49.6, 15.4)
- added J17: Conn_01x02_MountingPin, Connector_JST:JST_GH_SM02B-GHS-TB_1x02-1MP_P1.25mm_Horizontal, F.Cu at (16.8, 71.4)
- added J18: Conn_01x02_MountingPin, Connector_JST:JST_GH_SM02B-GHS-TB_1x02-1MP_P1.25mm_Horizontal, F.Cu at (16.9, 78.5)
- added J19: Conn_01x04_MountingPin, Connector_JST:JST_GH_BM04B-GHS-TBT_1x04-1MP_P1.25mm_Vertical, F.Cu at (16.6, 46.8)
- added J20: Conn_01x04, Connector_JST:JST_PH_B4B-PH-K_1x04_P2.00mm_Vertical, F.Cu at (15.1, 61.9)
- added J21: Conn_01x02, Connector_AMASS:AMASS_XT30PW-F_1x02_P2.50mm_Horizontal, F.Cu at (78.9, 21.2)
- added J28: SWD, Connector_Molex:Molex_PicoBlade_53261-0471_1x04-1MP_P1.25mm_Horizontal, F.Cu at (96.1, 106.9)
- added R85: 1k, Resistor_SMD:R_0603_1608Metric, F.Cu at (103.5, 88.3)
- added R86: 1k, Resistor_SMD:R_0603_1608Metric, F.Cu at (103.5, 97.8)
- added R87: 10k, Resistor_SMD:R_0603_1608Metric, F.Cu at (91.3, 100.7)
- added RN19: 82R, Resistor_SMD:R_Array_Concave_4x0603, F.Cu at (95.0, 101.0)
- C1, C109, C111, C112, C113, C114, C115, C116, C117, C118, C119, C14, C15, C19, C2, C21, C22, C23, C24, C25, C26, C28, C29, C3, C30, C31, C32, C33, C34, C35, C36, C37, C38, C39, C40, C41, C42, C43, C44, C45, C47, C48, C49, C50, C51, C53, C62, C63, C64, C65, C66, C67, C68, C69, C74, C75, C77, C78, C79, C80, C81, C82, C83, C84, C85, D13, D14, D16, D17, D18, D19, D20, D21, D3, D4, D5, J10, L2, L3, L7, R33, R34, R35, R36, R37, R38, R39, R40, R41, R42, R43, R44, R45, R67, R68, R69, R70, R71, R72, R73, R74, U10, U11, U17, U19, U3, U7, U8, U9: moved to B.Cu
- C101, C103, C105, C99, F2, Q1, Q2, U18: moved to F.Cu
- L1, L4, L5, L8: footprint Inductor_SMD:L_Changjiang_FXL1770 -> Inductor_SMD:L_Sunlord_MWSA0603S; moved to B.Cu
- moved J1 223.4 mm to (20.7, 90.7)
- moved J2 200.5 mm to (15.8, 28.7), turned to 90 degrees
- moved D11 190.0 mm to (15.1, 52.4)
- moved U16 185.7 mm to (27.1, 58.5), turned to 90 degrees
- moved D17 182.0 mm to (33.1, 80.1), turned to -90 degrees
- moved D18 181.7 mm to (31.2, 64.7), turned to -90 degrees
- moved U3 179.5 mm to (16.3, 46.9), turned to 90 degrees
- moved U6 179.5 mm to (19.8, 58.8), turned to 90 degrees
- moved J5 177.8 mm to (61.4, 15.7), turned to 180 degrees
- moved D4 176.6 mm to (28.3, 36.3)
- moved RN15 175.3 mm to (34.5, 28.6), turned to 90 degrees
- moved D9 173.2 mm to (49.6, 22.1), turned to 90 degrees
- moved RN13 171.3 mm to (30.7, 28.6), turned to 90 degrees
- moved J4 170.6 mm to (16.6, 37.3), turned to -90 degrees
- moved RN12 169.5 mm to (25.2, 35.0), turned to 180 degrees
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Connections:
- C47 pad 1: 7.4v_Servo -> +7.4v_Servo
- C49 pad 1: 7.4v_Servo -> +7.4v_Servo
- C82 pad 1: 7.4v_Servo -> +7.4v_Servo
- C83 pad 1: 7.4v_Servo -> +7.4v_Servo
- D20 pad 1: 7.4v_Servo -> +7.4v_Servo
- J4 pad 1: /MainControl/UART7_TX -> /MainControl/UART7_RX
- J4 pad 2: /MainControl/UART7_RX -> /MainControl/UART7_TX
- L5 pad 2: 7.4v_Servo -> +7.4v_Servo
- R46 pad 1: VOUT -> +24V
- R47 pad 1: VOUT -> +24V
- R71 pad 1: 7.4v_Servo -> +7.4v_Servo
- R84 pad 1: 7.4v_Servo -> +7.4v_Servo
- RN10 pad 3: /MainControl/PB14 -> /MainControl/PB15
- RN10 pad 4: /MainControl/PB15 -> /MainControl/PB14
- RN10 pad 5: /MainControl/UART4_CTS -> /MainControl/UART4_RTS
- RN10 pad 6: /MainControl/UART4_RTS -> /MainControl/UART4_CTS
- RN13 pad 1: /MainControl/PA7 -> /MainControl/PA4
- RN13 pad 2: /MainControl/PA6 -> /MainControl/PA5
- RN13 pad 3: /MainControl/PA5 -> /MainControl/PA7
- RN13 pad 4: /MainControl/PA4 -> /MainControl/PA6
- RN13 pad 5: /MainControl/CS_ICM-42688 -> /MainControl/SPI1_MISO
- RN13 pad 6: /MainControl/SPI1_SCK -> /MainControl/SPI1_MOSI
- RN13 pad 7: /MainControl/SPI1_MISO -> /MainControl/SPI1_SCK
- RN13 pad 8: /MainControl/SPI1_MOSI -> /MainControl/CS_ICM-42688
- RN6 pad 2: /MainControl/PD0 -> /MainControl/PD1
- RN6 pad 3: /MainControl/PD1 -> /MainControl/PD0
- RN6 pad 6: /MainControl/CAN1_TX -> /MainControl/CAN1_RX
- RN6 pad 7: /MainControl/CAN1_RX -> /MainControl/CAN1_TX
- RN7 pad 1: /MainControl/PA9 -> GND
- RN7 pad 4: GND -> /MainControl/PA9
- RN7 pad 5: GND -> /MainControl/UART1_TX
- RN7 pad 8: /MainControl/UART1_TX -> GND
- RN9 pad 1: /MainControl/PD8 -> /MainControl/PD12
- RN9 pad 3: /MainControl/PD12 -> /MainControl/PD8
- RN9 pad 6: /MainControl/UART2_DE -> /MainControl/UART3_TX
- RN9 pad 7: /MainControl/UART2_RX -> /MainControl/UART3_RX
- RN9 pad 8: /MainControl/UART2_TX -> /MainControl/UART3_DE
- U2 pad 13: /MainControl/IMU_SCLK -> /MainControl/SPI1_SCK
- U5 pad 6: /MainControl/RS422_TX+ -> /MainControl/RS422_TX-
- U6 pad 4: /MainControl/NUC2_DP -> /MainControl/NUC1_DP
Other:
- outline, holes or cut-outs redrawn

Commit message: update layout
Parts:
- removed RN19: 82R, Resistor_SMD:R_Array_Concave_4x0603
- C118, C119, C15: moved to F.Cu
- moved R84 143.1 mm to (25.4, 108.1), turned to 90 degrees
- moved D31 135.5 mm to (25.4, 105.1), turned to -90 degrees
- moved R78 117.8 mm to (105.2, 76.8)
- moved R80 113.7 mm to (25.9, 65.6), turned to 180 degrees
- moved R75 104.6 mm to (105.1, 73.9)
- moved D27 103.2 mm to (22.9, 65.6)
- moved D25 92.7 mm to (108.2, 76.8), turned to 180 degrees
- moved D30 91.2 mm to (13.7, 23.4)
- moved D29 89.4 mm to (20.7, 30.7), turned to -90 degrees
- moved D22 88.0 mm to (108.1, 73.9), turned to 180 degrees
- moved R82 87.1 mm to (20.6, 33.7), turned to 90 degrees
- moved R79 86.4 mm to (78.5, 50.2)
- moved D28 83.0 mm to (21.2, 15.1), turned to -90 degrees
- moved R83 81.6 mm to (16.6, 23.4), turned to 180 degrees
- moved R81 77.8 mm to (21.2, 18.1), turned to 90 degrees
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Connections:
- J11 pad 1: /MainControl/CAN1_H -> /MainControl/CAN1_L
- J11 pad 2: /MainControl/CAN1_L -> /MainControl/CAN1_H
- J12 pad 1: /MainControl/CAN1_H -> /MainControl/CAN1_L
- J12 pad 2: /MainControl/CAN1_L -> /MainControl/CAN1_H
- J3 pad 1: /MainControl/Pul+ -> /MainControl/Dir-
- J3 pad 2: /MainControl/Pul- -> /MainControl/Dir+
- J3 pad 3: /MainControl/Dir+ -> /MainControl/Pul-
- J3 pad 4: /MainControl/Dir- -> /MainControl/Pul+
- RN12 pad 1: /MainControl/PE8 -> GND
- RN12 pad 2: /MainControl/PE7 -> GND
- RN12 pad 3: GND -> /MainControl/PE8
- RN12 pad 4: GND -> /MainControl/PE7
- RN12 pad 5: GND -> /MainControl/UART7_RX
- RN12 pad 6: GND -> /MainControl/UART7_TX
- RN12 pad 7: /MainControl/UART7_RX -> GND
- RN12 pad 8: /MainControl/UART7_TX -> GND
- RN14 pad 1: /MainControl/PE0 -> /MainControl/PE1
- RN14 pad 2: /MainControl/PE1 -> /MainControl/PE0
- RN14 pad 7: /MainControl/UART8_RX -> /MainControl/UART8_TX
- RN14 pad 8: /MainControl/UART8_TX -> /MainControl/UART8_RX
- RN18 pad 6: /MainControl/TIM2_CH3 -> /MainControl/TIM4_CH3
- RN18 pad 8: /MainControl/TIM2_CH4 -> /MainControl/TIM4_CH4
- RN6 pad 1: GND -> /MainControl/PD1
- RN6 pad 2: /MainControl/PD1 -> /MainControl/PD0
- RN6 pad 3: /MainControl/PD0 -> /MainControl/PA14
- RN6 pad 4: GND -> /MainControl/PA13
- RN6 pad 5: GND -> /MainControl/SWD_DIO
- RN6 pad 6: /MainControl/CAN1_RX -> /MainControl/SWD_CLK
- RN6 pad 7: /MainControl/CAN1_TX -> /MainControl/CAN1_RX
- RN6 pad 8: GND -> /MainControl/CAN1_TX
Routing:
- net +5V: track 0.00 -> 231.7 mm, vias 0 -> 168
- net +3.3V_MCU: track 0.00 -> 171.9 mm, vias 0 -> 114
- net +3.3V_IO: track 0.00 -> 164.9 mm, vias 0 -> 81
- net /MainControl/NRST: track 0.00 -> 66.7 mm, vias 0 -> 2
- net /MainControl/PB10: track 0.00 -> 64.8 mm, vias 0 -> 2
- net /MainControl/PB11: track 0.00 -> 62.0 mm, vias 0 -> 2
- net /MainControl/BOOT0: track 0.00 -> 58.1 mm
- net /Power/VAUX: track 0.00 -> 55.9 mm, vias 0 -> 4
- net +24V: track 0.00 -> 54.7 mm, vias 0 -> 1
- net /Power/VCC: track 0.00 -> 47.7 mm, vias 0 -> 8
- net /MainControl/PE0: track 0.00 -> 46.4 mm
- net /MainControl/PE1: track 0.00 -> 45.9 mm
- net /MainControl/PD14: track 0.00 -> 43.2 mm, vias 0 -> 2
- net /MainControl/PD15: track 0.00 -> 41.5 mm, vias 0 -> 2
- net /MainControl/PD2: track 0.00 -> 40.5 mm, vias 0 -> 2
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- added copper zone on B.Cu, net +12V_Motor
- added copper zone on B.Cu, net +24V
- added copper zone on F.Cu, net +24V
- added copper zone on B.Cu, net +3.3V_IO
- added copper zone on F.Cu, net +3.3V_IO
- added copper zone on In2.Cu, net +3.3V_IO
- added copper zone on B.Cu, net +3.3V_MCU
- added copper zone on F.Cu, net +3.3V_MCU
- added copper zone on In2.Cu, net +3.3V_MCU
- added copper zone on B.Cu, net +3.3V_SatellieCom
- added copper zone on F.Cu, net +3.3V_SatellieCom
- added copper zone on B.Cu, net +48V
- added copper zone on F.Cu, net +48V
- added copper zone on B.Cu, net +5V
- added copper zone on F.Cu, net +5V
- added copper zone on In2.Cu, net +5V
- added copper zone on B.Cu, net +5V_SatellieCom
- added copper zone on B.Cu, net +7.4v_Servo
- added copper zone on F.Cu, net /Power/SW
- added copper zone on F.Cu, net /Power/VAUX
- added copper zone on F.Cu, net /Power/VCC
- added copper zone on B.Cu, net GND
- added copper zone on F.Cu, net GND
- added copper zone on In1.Cu, net GND
- added copper zone on In2.Cu, net GND
- added copper zone on B.Cu, net Net-(D14-K)
- added copper zone on B.Cu, net Net-(D3-K)
- added copper zone on B.Cu, net Net-(D4-K)
- added copper zone on B.Cu, net Net-(D5-K)
- added copper zone on F.Cu, net Net-(J10-Pin_2)
- added copper zone on F.Cu, net Net-(Q1-D)
- added copper zone on F.Cu, net Net-(U12-LX)
- added copper zone on B.Cu, net Net-(U17-SW)
Other:
- outline, holes or cut-outs redrawn
- copper layers 2 -> 4
- board text added: "- +"
- board text added: "- DP DN +"
- board text added: "24V PWR"
- board text added: "48V PWR IN"
- board text added: "5V"
- board text added: "A"
- board text added: "B"
- board text added: "BOOT0"
- board text added: "CAN1"
- board text added: "DIO CLK GND 3V3"
- board text added: "H"
- board text added: "L"
- board text added: "Motor 12V"
- board text added: "NRST"
- board text added: "PWR In 48v"
- board text added: "Powered by STM32H743"
- board text added: "Pul+ - Dir+ -"
- board text added: "RS422 UART5"
- board text added: "RS485 UART1"
- board text added: "RS485 UART2"
- board text added: "RS485 UART3"
- board text added: "RX 5V GND"
- board text added: "RX TX 3V3 GND"
- board text added: "SBUS UART8"
- board text added: "SD Card"
- board text added: "SWD"
- board text added: "SatellieCom UART7"
- board text added: "SatelliePWR 5V"
- board text added: "Servo Motor PWM 7.4V -"
- board text added: "Stepper"
- board text added: "T+ T- R- R+"
- board text added: "T2C4 T4C4 T2C3 T4C3"
- board text added: "USB-TTL"
- board text added: "UnderwaterGlider V0.1 By OU,Farui Contact:fou @ust.hk"

Commit message: update version,submit custom
Parts:
- moved J18 3.30 mm to (13.7, 79.2)
- moved J17 3.27 mm to (13.7, 72.2)
- moved R82 3.20 mm to (17.6, 32.8)
- moved J19 3.15 mm to (13.5, 46.3)
- moved R22 3.15 mm to (15.0, 51.9)
- moved D11 3.15 mm to (12.0, 51.9)
- moved J4 2.99 mm to (13.6, 36.8)
- moved D29 2.53 mm to (19.1, 32.8), turned to 90 degrees
- moved J20 2.51 mm to (12.7, 61.1)
- moved J3 2.40 mm to (68.7, 13.2)
- moved J5 2.38 mm to (61.4, 13.3)
- moved D24 2.35 mm to (56.1, 11.6)
- moved R77 2.35 mm to (56.1, 14.6)
- moved J15 1.86 mm to (42.8, 13.6)
- moved J16 1.86 mm to (49.8, 13.6)
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Routing:
- net /MainControl/RS422_RX+: track 7.81 -> 21.9 mm
- net /MainControl/UART4_CTS: track 22.5 -> 27.0 mm
- net /MainControl/NUC1_ACT: track 15.8 -> 19.1 mm
- net /MainControl/UART7_TX: track 5.85 -> 9.01 mm
- net /MainControl/UART7_RX: track 6.04 -> 9.19 mm
- net /MainControl/RS422_RX-: track 7.81 -> 11.0 mm
- net /MainControl/RS422_TX-: track 7.82 -> 11.0 mm
- net /MainControl/RS422_TX+: track 7.83 -> 10.9 mm
- net +3.3V_IO: track 164.9 -> 167.9 mm
- net /MainControl/RS485_Bus3_A: track 21.7 -> 24.5 mm
- net /MainControl/RS485_Bus3_B: track 22.5 -> 25.2 mm
- net /MainControl/Pul-: track 8.78 -> 11.2 mm
- net /MainControl/Dir+: track 8.97 -> 11.4 mm
- net /MainControl/Pul+: track 8.60 -> 11.0 mm
- net /MainControl/Dir-: track 9.87 -> 12.2 mm
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